Commit message: fix: resolve RViz2 robot model and image display issues (performed by Claude)
- Remove leading slash from TF child frame ("/bluerov/base_link" -> "bluerov/base_link")
  so RViz2 can match the TF broadcast to the URDF link name
- Fix URDF mesh package path (ORB_DVL2 -> aqua_slam) so robot_state_publisher
  can locate the BlueROV2 mesh at runtime
- Set image header stamp and frame_id in PublishImgWithInfo so RViz2 accepts
  the image stream instead of showing "No Image"
- Update rviz config for ROS2 Jazzy: rename Image Topic->Topic, replace
  Robot Description with Description Source/Topic, remove Transport Hint
  (property no longer exists in Jazzy)

File: urdf/bluerov.urdf (robot description, URDF)
Before this commit: robot vehicle, 1 links, 0 joints
Links:
- link bluerov/base_link: geometry visual mesh filename=package://aqua_slam/urdf/bluerov2_noprop.dae scale=1 1 1
